File: ECAD IOT SMART SWITCH/IOT SMART SWITCH/IOT SMART SWITCH.sch (KiCad schematic (older format))
At the start: 31 parts

Commit message: work in progress
Parts:
- added C6, C8: C, symbol pspice:C
- added D6, D7, D8: LED, symbol Device:LED
- added R10, R11, R12, R13, R3, R7: R, symbol Device:R
- added U3: LM317_TO39, Package_TO_SOT_THT:TO-39-3, symbol Regulator_Linear:LM317_TO39
- gave numbers to parts that had none: 31
Connections:
- net 10V_DC: now also C6.1, U3.1 (VI)
- net 5V_DC: no longer C7.1, J5.20 (Pin_20), R4.1, R5.1, R8.1, T2.4, U2.3 (VO)
- net ESP_Pin_21: now also J4.11 (Pin_11); no longer J4.14 (Pin_14)
- net GND: now also J4.20 (Pin_20), C6.2, C8.2, R11.2, R12.2, R13.2, R7.2; no longer J5.15 (Pin_15)
- net at R2.1, U1.3: now also R3.2; no longer M1.2 (G)
- net 3V3_DC: now reaches J5.2 (Pin_2)
- net 3V3_DC: now also R4.1, R5.1, T2.4, C8.1, D8.2 (A), R10.1, U3.3 (VO)
- new net: M1.2 (G), R3.1
- new net: R10.2, R11.1, U3.2 (ADJ)
- new net: D8.1 (K), R13.1
- new net: D7.1 (K), R12.1
- new net: D6.1 (K), R7.1
- new net 12V_DC: C7.1, D7.2 (A), R8.1, U2.3 (VO)
Other:
- moved on the sheet: J4, J5

Commit message: Associations are tough
Parts:
- removed U1: SFH617A-1, Package_DIP:DIP-4_W7.62mm, symbol Isolator:SFH617A-1
- added U1: 4N25, Package_DIP:DIP-6_W7.62mm, symbol Isolator:4N25
- C1: value C -> 100u
- C2: value C -> 100p
- C3: value C -> 10u
- C4, C7, C8: value C -> 1u
- C5, C6: value C -> 0.1u
- D1, D2, D3, D4, D5: value DIODE -> 1N5822; footprint (none) -> Diode_THT:D_DO-201AD_P15.24mm_Horizontal
- K1: footprint Relay_THT:Relay_SPDT_SANYOU_SRD_Series_Form_C -> SLA-12VDC-SL-C:SLA12VDCSLC
- R1, R10, R2, R3, R4, R5, R8: value R -> 1k
- R11: value R -> 1.6k
- R12, R13: value R -> 10k
- R6: value R -> 800R
- R9: value R -> 9.1k
- T1: value Transformer_1P_1S -> VC 10/1/18
- T2: value CST1 -> AC1020
Connections:
- net labels added: -18V_AC, 16V_DC
- net labels removed: -12V_AC, 10V_DC, 5V_DC
Other:
- moved on the sheet: C1, C3, C4, C5, C6, C7, C8, D2, D3, D4, D5, D6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
