File: ECAD IOT SMART SWITCH/IOT SMART SWITCH/IOT SMART SWITCH.sch (KiCad schematic (older format))
At the start: 43 parts, among them J1 Conn_02x02_Odd_Even, J2 Conn_02x02_Odd_Even, J3 Conn_02x02_Odd_Even, J4 Conn_01x20, J5 Conn_01x20, J6 Conn_02x02_Odd_Even, J7 Conn_02x02_Odd_Even, K1 SLA-12VDC-SL, Q1 BS170, T1 VC 10/1/18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

Commit message: Associate last pieces
Parts:
- removed C8: 1u, symbol pspice:C
- removed J4, J5: Conn_01x20, symbol Connector_Generic:Conn_01x20
- added J4, J5: Conn_01x16, Connector_PinSocket_2.54mm:PinSocket_1x16_P2.54mm_Vertical, symbol Connector_Generic:Conn_01x16
- C1: value 100u -> 220u; footprint (none) -> Capacitor_THT:CP_Radial_D6.3mm_P2.50mm
- C2: footprint (none) -> Capacitor_THT:CP_Radial_D5.0mm_P2.00mm
- C3: value 10u -> 100u; footprint (none) -> Capacitor_THT:CP_Radial_D5.0mm_P2.00mm
- C4, C7: value 1u -> 10u; footprint (none) -> Capacitor_THT:CP_Radial_D5.0mm_P2.00mm
- C5, C6: value 0.1u -> 10u; footprint (none) -> Capacitor_THT:CP_Radial_D5.0mm_P2.00mm
- D6, D7, D8: footprint (none) -> LED_THT:LED_D3.0mm
- R1, R10, R11, R12, R13, R2, R3, R4, R5, R6, R7, R8, R9: footprint (none) -> Resistor_SMD:R_1020_2550Metric_Pad1.33x5.20mm_HandSolder
Connections:
- net labels added: CT_ADC, GNDPWR
- net labels removed: GND, MAINS_L_Output, MAINS_N_Output
- wire segments 151 -> 142
- no-connect marks 1 -> 31
Other:
- moved on the sheet: D6, J6, R1, R7

Commit message: PCB New Start
Parts:
- U2, U3: footprint Package_TO_SOT_THT:TO-39-3 -> LM317T_XT:TO255P460X1020X2008-3P
Connections:
- no-connect marks 31 -> 30
Changed lines of the file:
@@
 F 0 "U2" H 8900 1192 50  0000 C CNN
 F 1 "LM317_TO39" H 8900 1101 50  0000 C CNN
-F 2 "Package_TO_SOT_THT:TO-39-3" H 8900 1175 50  0001 C CIN
+F 2 "LM317T_XT:TO255P460X1020X2008-3P" H 8900 1175 50  0001 C CIN
 F 3 "http://www.ti.com/lit/ds/symlink/lm317.pdf" H 8900 950 50  0001 C CNN
 	1    8900 950
@@
 Wire Wire Line
 	1750 1700 1750 1800
-NoConn ~ 1750 1750
 Wire Wire Line
 	1300 2600 1300 2700
@@
 	6450 7100 6450 7350
 Wire Wire Line
-	6450 7350 6300 7350
-Wire Wire Line
-	6300 7450 6300 7350
-Connection ~ 6300 7350
-Wire Wire Line
 	5350 6700 5350 6000
 Text GLabel 8400 5200 2    50   Input ~ 0
@@
 Wire Wire Line
 	6100 7350 6100 7300
-Wire Wire Line
-	6100 7350 6300 7350
 Wire Wire Line
 	6100 6800 6100 6700
@@
 F 0 "U3" H 9000 2592 50  0000 C CNN
 F 1 "LM317_TO39" H 9000 2501 50  0000 C CNN
-F 2 "Package_TO_SOT_THT:TO-39-3" H 9000 2575 50  0001 C CIN
+F 2 "LM317T_XT:TO255P460X1020X2008-3P" H 9000 2575 50  0001 C CIN
 F 3 "http://www.ti.com/lit/ds/symlink/lm317.pdf" H 9000 2350 50  0001 C CNN
 	1    9000 2350
@@
 L power:GNDPWR #PWR0103
 U 1 1 60F2B189
-P 2050 6450
-F 0 "#PWR0103" H 2050 6250 50  0001 C CNN
-F 1 "GNDPWR" H 2054 6296 50  0000 C CNN
-F 2 "" H 2050 6400 50  0001 C CNN
-F 3 "" H 2050 6400 50  0001 C CNN
-	1    2050 6450
+P 2050 6500
+F 0 "#PWR0103" H 2050 6300 50  0001 C CNN
+F 1 "GNDPWR" H 2054 6346 50  0000 C CNN
+F 2 "" H 2050 6450 50  0001 C CNN
+F 3 "" H 2050 6450 50  0001 C CNN
+	1    2050 6500
 	1    0    0    -1
 $EndComp
@@
 L power:GNDPWR #PWR0107
 U 1 1 60F2E4F2
-P 6300 7450
-F 0 "#PWR0107" H 6300 7250 50  0001 C CNN
-F 1 "GNDPWR" H 6304 7296 50  0000 C CNN
-F 2 "" H 6300 7400 50  0001 C CNN
-F 3 "" H 6300 7400 50  0001 C CNN
-	1    6300 7450
+P 6300 7350
+F 0 "#PWR0107" H 6300 7150 50  0001 C CNN
+F 1 "GNDPWR" H 6304 7196 50  0000 C CNN
+F 2 "" H 6300 7300 50  0001 C CNN
+F 3 "" H 6300 7300 50  0001 C CNN
+	1    6300 7350
 	1    0    0    -1
 $EndComp
@@
 Wire Wire Line
 	10000 3350 10000 3500
+Wire Wire Line
+	6100 7350 6300 7350
+Connection ~ 6300 7350
+Wire Wire Line
+	6300 7350 6450 7350
+Wire Wire Line
+	2050 6500 2050 6450
 $EndSCHEMATC
