File: ECAD IOT SMART SWITCH/IOT SMART SWITCH/IOT SMART SWITCH.sch (KiCad schematic (older format))
At the start: 43 parts, among them J4 Conn_01x16, J5 Conn_01x16, K1 SLA-12VDC-SL-C, Q1 BS170, T1 VC_10_1_18, T2 AC-1020, U1 4N25, U2 LM317_TO39, U3 LM317_TO39

Commit message: then go run after it
Parts:
- gave numbers to parts that had none: 6
Connections:
- net 16V_DC: no longer U3.1 (VI)
Changed lines of the file:
@@
 	7800 1950 9400 1950
-Wire Wire Line
-	7900 2350 8700 2350
 Wire Wire Line
 	9400 1950 9950 1950
@@
 NoConn ~ 4300 5100
 $Comp
-L KF301-2P:KF301-2P J?
+L KF301-2P:KF301-2P J2
 U 1 1 60C9A2D8
 P 1800 1750
-F 0 "J?" H 2092 1385 50  0000 C CNN
+F 0 "J2" H 2092 1385 50  0000 C CNN
 F 1 "KF301-2P" H 2092 1476 50  0000 C CNN
 F 2 "KF3012P" H 2450 1850 50  0001 L CNN
@@
 $EndComp
 $Comp
-L KF301-2P:KF301-2P J?
+L KF301-2P:KF301-2P J1
 U 1 1 60C9A796
 P 1800 850
-F 0 "J?" H 2092 485 50  0000 C CNN
+F 0 "J1" H 2092 485 50  0000 C CNN
 F 1 "KF301-2P" H 2092 576 50  0000 C CNN
 F 2 "KF3012P" H 2450 950 50  0001 L CNN
@@
 $EndComp
 $Comp
-L KF301-2P:KF301-2P J?
+L KF301-2P:KF301-2P J7
 U 1 1 60CA1AAA
 P 10550 5050
-F 0 "J?" H 10950 5300 50  0000 C CNN
+F 0 "J7" H 10950 5300 50  0000 C CNN
 F 1 "KF301-2P" H 10950 5200 50  0000 C CNN
 F 2 "KF3012P" H 11200 5150 50  0001 L CNN
@@
 $EndComp
 $Comp
-L KF301-2P:KF301-2P J?
+L KF301-2P:KF301-2P J6
 U 1 1 60CA1E3D
 P 10500 6250
-F 0 "J?" H 10900 6500 50  0000 C CNN
+F 0 "J6" H 10900 6500 50  0000 C CNN
 F 1 "KF301-2P" H 10900 6400 50  0000 C CNN
 F 2 "KF3012P" H 11150 6350 50  0001 L CNN
@@
 $EndComp
 $Comp
-L KF301-2P:KF301-2P J?
+L KF301-2P:KF301-2P J3
 U 1 1 60C97AA0
 P 1800 2700
-F 0 "J?" H 2092 2335 50  0000 C CNN
+F 0 "J3" H 2092 2335 50  0000 C CNN
 F 1 "KF301-2P" H 2092 2426 50  0000 C CNN
 F 2 "KF3012P" H 2450 2800 50  0001 L CNN
@@
 Connection ~ 10500 6300
 $Comp
-L KF301-2P:KF301-2P J?
+L KF301-2P:KF301-2P J8
 U 1 1 60D01CDA
 P 10550 5650
-F 0 "J?" H 10950 5900 50  0000 C CNN
+F 0 "J8" H 10950 5900 50  0000 C CNN
 F 1 "KF301-2P" H 10950 5800 50  0000 C CNN
 F 2 "KF3012P" H 11200 5750 50  0001 L CNN

Commit message: Kicad project done for now
Parts:
- removed T2: AC-1020, AC-1020:AC1015, symbol IOT-SMART-SWITCH-rescue:AC-1020-AC-1020
- added T2: AC-1020, AC1015, symbol AC-1020:AC-1020
- J1, J2, J3, J6, J7, J8: symbol KF301-2P:KF301-2P -> IOT-SMART-SWITCH-rescue:KF301-2P-KF301-2P
Connections:
- net 16V_DC: now also U3.1 (VI)
- net CT_ADC: now also T2.1
- net at C2.1, R4.2, R5.2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: now also T2.2
Changed lines of the file:
@@
 EESchema Schematic File Version 4
 LIBS:IOT SMART SWITCH-cache
-EELAYER 30 0
+EELAYER 26 0
 EELAYER END
 $Descr A4 11693 8268
@@
 Text GLabel 10650 2350 2    50   Input ~ 0
 3V3_DC
-Text GLabel 7900 2350 0    50   Input ~ 0
+Text GLabel 8700 2350 0    50   Input ~ 0
 16V_DC
 $Comp
@@
 Wire Wire Line
 	4050 1850 4300 1850
-$Comp
-L IOT-SMART-SWITCH-rescue:AC-1020-AC-1020 T2
-U 1 1 60D00784
-P 5300 6200
-F 0 "T2" H 5700 6465 50  0000 C CNN
-F 1 "AC-1020" H 5700 6374 50  0000 C CNN
-F 2 "AC-1020:AC1015" H 5950 6300 50  0001 L CNN
-F 3 "http://docs-asia.electrocomponents.com/webdocs/0776/0900766b807760fc.pdf" H 5950 6200 50  0001 L CNN
-F 4 "PCB Mount Current Transformer" H 5950 6100 50  0001 L CNN "Description"
-F 5 "23" H 5950 6000 50  0001 L CNN "Height"
-F 6 "Nuvotem Talema" H 5950 5900 50  0001 L CNN "Manufacturer_Name"
-F 7 "AC-1020" H 5950 5800 50  0001 L CNN "Manufacturer_Part_Number"
-F 8 "" H 5950 5700 50  0001 L CNN "Mouser Part Number"
-F 9 "" H 5950 5600 50  0001 L CNN "Mouser Price/Stock"
-F 10 "" H 5950 5500 50  0001 L CNN "Arrow Part Number"
-F 11 "" H 5950 5400 50  0001 L CNN "Arrow Price/Stock"
-	1    5300 6200
-	1    0    0    -1
-$EndComp
 Wire Wire Line
 	6100 6300 6100 6900
@@
 NoConn ~ 4300 5100
 $Comp
-L KF301-2P:KF301-2P J2
+L IOT-SMART-SWITCH-rescue:KF301-2P-KF301-2P J2
 U 1 1 60C9A2D8
 P 1800 1750
@@
 $EndComp
 $Comp
-L KF301-2P:KF301-2P J1
+L IOT-SMART-SWITCH-rescue:KF301-2P-KF301-2P J1
 U 1 1 60C9A796
 P 1800 850
@@
 $EndComp
 $Comp
-L KF301-2P:KF301-2P J7
+L IOT-SMART-SWITCH-rescue:KF301-2P-KF301-2P J7
 U 1 1 60CA1AAA
 P 10550 5050
@@
 $EndComp
 $Comp
-L KF301-2P:KF301-2P J6
+L IOT-SMART-SWITCH-rescue:KF301-2P-KF301-2P J6
 U 1 1 60CA1E3D
 P 10500 6250
@@
 $EndComp
 $Comp
-L KF301-2P:KF301-2P J3
+L IOT-SMART-SWITCH-rescue:KF301-2P-KF301-2P J3
 U 1 1 60C97AA0
 P 1800 2700
@@
 Connection ~ 10500 6300
 $Comp
-L KF301-2P:KF301-2P J8
+L IOT-SMART-SWITCH-rescue:KF301-2P-KF301-2P J8
 U 1 1 60D01CDA
 P 10550 5650
@@
 Text GLabel 1800 1700 2    50   Input ~ 0
 Earth
+$Comp
+L AC-1020:AC-1020 T2
+U 1 1 60CA602E
+P 5300 6200
+F 0 "T2" H 5700 6465 50  0000 C CNN
+F 1 "AC-1020" H 5700 6374 50  0000 C CNN
+F 2 "AC1015" H 5950 6300 50  0001 L CNN
+F 3 "http://docs-asia.electrocomponents.com/webdocs/0776/0900766b807760fc.pdf" H 5950 6200 50  0001 L CNN
+F 4 "PCB Mount Current Transformer" H 5950 6100 50  0001 L CNN "Description"
+F 5 "23" H 5950 6000 50  0001 L CNN "Height"
+F 6 "Nuvotem Talema" H 5950 5900 50  0001 L CNN "Manufacturer_Name"
+F 7 "AC-1020" H 5950 5800 50  0001 L CNN "Manufacturer_Part_Number"
+F 8 "" H 5950 5700 50  0001 L CNN "Mouser Part Number"
+F 9 "" H 5950 5600 50  0001 L CNN "Mouser Price/Stock"
+F 10 "" H 5950 5500 50  0001 L CNN "Arrow Part Number"
+F 11 "" H 5950 5400 50  0001 L CNN "Arrow Price/Stock"
+	1    5300 6200
+	1    0    0    -1
+$EndComp
 $EndSCHEMATC

Commit message: RE-Think Things
Parts:
- J1, J2, J3, J6, J7, J8: symbol IOT-SMART-SWITCH-rescue:KF301-2P-KF301-2P -> IOT-SMART-SWITCH-rescue:KF301-2P-KF301-2P-IOT-SMART-SWITCH-rescue
- T2: symbol AC-1020:AC-1020 -> IOT-SMART-SWITCH-rescue:AC-1020-AC-1020
Changed lines of the file:
@@
 EESchema Schematic File Version 4
 LIBS:IOT SMART SWITCH-cache
-EELAYER 26 0
+EELAYER 30 0
 EELAYER END
 $Descr A4 11693 8268
@@
 NoConn ~ 4300 5100
 $Comp
-L IOT-SMART-SWITCH-rescue:KF301-2P-KF301-2P J2
+L IOT-SMART-SWITCH-rescue:KF301-2P-KF301-2P-IOT-SMART-SWITCH-rescue J2
 U 1 1 60C9A2D8
 P 1800 1750
@@
 $EndComp
 $Comp
-L IOT-SMART-SWITCH-rescue:KF301-2P-KF301-2P J1
+L IOT-SMART-SWITCH-rescue:KF301-2P-KF301-2P-IOT-SMART-SWITCH-rescue J1
 U 1 1 60C9A796
 P 1800 850
@@
 $EndComp
 $Comp
-L IOT-SMART-SWITCH-rescue:KF301-2P-KF301-2P J7
+L IOT-SMART-SWITCH-rescue:KF301-2P-KF301-2P-IOT-SMART-SWITCH-rescue J7
 U 1 1 60CA1AAA
 P 10550 5050
@@
 $EndComp
 $Comp
-L IOT-SMART-SWITCH-rescue:KF301-2P-KF301-2P J6
+L IOT-SMART-SWITCH-rescue:KF301-2P-KF301-2P-IOT-SMART-SWITCH-rescue J6
 U 1 1 60CA1E3D
 P 10500 6250
@@
 $EndComp
 $Comp
-L IOT-SMART-SWITCH-rescue:KF301-2P-KF301-2P J3
+L IOT-SMART-SWITCH-rescue:KF301-2P-KF301-2P-IOT-SMART-SWITCH-rescue J3
 U 1 1 60C97AA0
 P 1800 2700
@@
 Connection ~ 10500 6300
 $Comp
-L IOT-SMART-SWITCH-rescue:KF301-2P-KF301-2P J8
+L IOT-SMART-SWITCH-rescue:KF301-2P-KF301-2P-IOT-SMART-SWITCH-rescue J8
 U 1 1 60D01CDA
 P 10550 5650
@@
 Earth
 $Comp
-L AC-1020:AC-1020 T2
+L IOT-SMART-SWITCH-rescue:AC-1020-AC-1020 T2
 U 1 1 60CA602E
 P 5300 6200
