File: ECAD IOT SMART SWITCH/IOT SMART SWITCH/IOT SMART SWITCH.kicad_pcb (KiCad board)
At the start: 2 copper layers, 42 parts, among them J1 Conn_02x02_Odd_Even, J2 Conn_02x02_Odd_Even, J3 Conn_02x02_Odd_Even, J4 Conn_01x16, J5 Conn_01x16, J6 Conn_02x02_Odd_Even, J7 Conn_02x02_Odd_Even, K1 SLA-12VDC-SL, Q1 BS170, T1 VC 10/1/18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

Commit message: eeschema updated
Parts:
- D2, D3, D4, D5: value 1N5822 -> 1N5822
- K1: value SLA-12VDC-SL -> SLA-12VDC-SL-C
- R1, R10, R11, R12, R13, R2, R3, R5, R6, R7, R8, R9: footprint Resistor_SMD:R_1020_2550Metric_Pad1.33x5.20mm_HandSolder -> Resistor_SMD:R_1206_3216Metric
- R4: value 1k -> 50; footprint Resistor_SMD:R_1020_2550Metric_Pad1.33x5.20mm_HandSolder -> Resistor_SMD:R_1206_3216Metric
- T1: value VC 10/1/18 -> VC_10_1_18
- T2: value AC1020 -> AC-1020
- moved R5 82.9 mm to (217.0, 68.6)
- moved D1 65.6 mm to (138.4, 90.2)
- moved D8 62.6 mm to (186.7, 118.1)
- moved R11 60.2 mm to (171.4, 118.1), turned to 90 degrees
- moved R6 53.7 mm to (217.2, 76.2), turned to 180 degrees
- moved R1 52.2 mm to (162.6, 90.0), turned to 270 degrees
- moved D7 50.6 mm to (186.7, 109.2)
- moved J5 49.8 mm to (167.6, 102.9), turned to 270 degrees
- moved J7 49.5 mm to (184.2, 64.8)
- moved C2 49.3 mm to (208.3, 68.6)
- moved R8 45.5 mm to (179.1, 109.3), turned to 270 degrees
- moved C6 44.9 mm to (163.8, 113.0)
- moved R2 44.3 mm to (196.8, 92.7)
- moved J2 43.2 mm to (112.7, 47.0), turned to 0 degrees
- moved J3 41.7 mm to (77.1, 46.6), turned to 180 degrees
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Connections:
- D2 pad 1: Net-(D2-Pad1) -> 16V_DC
- D2 pad 2: 16V_DC -> Net-(D2-Pad2)
- D3 pad 1: GNDPWR -> Net-(D2-Pad2)
- D3 pad 2: Net-(D2-Pad1) -> GNDPWR
- D4 pad 1: -18V_AC -> 16V_DC
- D4 pad 2: 16V_DC -> -18V_AC
- D5 pad 1: GNDPWR -> -18V_AC
- D5 pad 2: -18V_AC -> GNDPWR
- K1 pad 2: Net-(D1-Pad1) -> 12V_DC
- K1 pad 5: 12V_DC -> Net-(J7-Pad1)
- K1 pad 6: (no net) -> Net-(D1-Pad1)
- T1 pad 4: Net-(D2-Pad1) -> -18V_AC
- T1 pad 5: (no net) -> Net-(D2-Pad2)
- T1 pad 6: (no net) -> Net-(D2-Pad2)
- T2 pad 1: Net-(T2-Pad1) -> CT_ADC
- T2 pad 2: Net-(T2-Pad2) -> Net-(C2-Pad1)

Commit message: Is fridge running
Parts:
- added J8: KF301-2P, KF3012P, F.Cu at (204.5, 44.7)
- J1, J2, J3, J6, J7: value Conn_02x02_Odd_Even -> KF301-2P; footprint KF301-2P:KF3012P -> KF3012P
- moved Q1 60.8 mm to (135.1, 80.8)
- moved R3 59.0 mm to (146.2, 80.5)
- moved J2 34.0 mm to (78.7, 45.7)
- moved R2 27.9 mm to (208.4, 118.1), turned to 180 degrees
- moved C5 22.9 mm to (190.5, 83.8)
- moved J4 22.9 mm to (190.5, 77.5)
- moved J5 22.9 mm to (190.5, 102.9)
- moved R13 22.3 mm to (200.7, 122.0)
- moved R1 21.8 mm to (184.3, 88.4), turned to 0 degrees
- moved J3 20.9 mm to (98.0, 45.7), turned to 0 degrees
- moved J6 19.9 mm to (191.0, 44.7)
- moved J1 19.7 mm to (117.5, 45.7), turned to 0 degrees
- moved U1 16.1 mm to (202.2, 88.4), turned to 0 degrees
- moved J7 15.0 mm to (169.7, 60.7)
- moved T2 13.3 mm to (172.2, 46.7)
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Connections:
- J1 pad 1: Net-(J1-Pad1) -> MAINS_L
- J1 pad 2: Net-(J1-Pad2) -> MAINS_L
- J2 pad 1: Net-(J2-Pad1) -> Earth
- J2 pad 2: MAINS_L -> Earth
- J3 pad 1: Net-(J3-Pad1) -> MAINS_N
- J6 pad 2: Net-(J6-Pad2) -> MAINS_N
- J7 pad 2: Net-(J7-Pad2) -> Net-(J7-Pad1)
Routing:
- net GNDPWR: track 0.00 -> 377.7 mm, vias 0 -> 4
- net 3V3_DC: track 0.00 -> 186.4 mm, vias 0 -> 2
- net Earth: track 0.00 -> 138.3 mm
- net MAINS_N: track 0.00 -> 133.7 mm
- net 12V_DC: track 0.00 -> 113.9 mm
- net CT_ADC: track 0.00 -> 113.3 mm, vias 0 -> 2
- net Net-(R2-Pad1): track 0.00 -> 96.7 mm
- net 16V_DC: track 0.00 -> 90.1 mm
- net Net-(R8-Pad2): track 0.00 -> 71.7 mm
- net Net-(C2-Pad1): track 0.00 -> 69.9 mm
- net MAINS_L: track 0.00 -> 61.9 mm
- net Net-(R10-Pad2): track 0.00 -> 58.6 mm
- net Net-(D6-Pad2): track 0.00 -> 47.9 mm
- net Net-(J7-Pad1): track 0.00 -> 43.8 mm
- net -18V_AC: track 0.00 -> 32.4 mm
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Other:
- board outline added: 156.2 x 92.7 mm
- net class HV_NET added: clearance 4, trace_width 2, via_dia 0.8, via_drill 0.4

Commit message: Ready for quotes
Parts:
- moved J8 0.40 mm to (204.9, 44.8)
Routing:
- net 12V_DC: track 113.9 -> 154.8 mm, vias 0 -> 3
- net GNDPWR: track 377.7 -> 381.6 mm
- net Net-(R10-Pad2): track 58.6 -> 62.0 mm
- added copper zone on B.Cu, net Earth
- added copper zone on F.Cu, net Earth
Other:
- outline, holes or cut-outs redrawn

Commit message: RE-Think Things
Other:
- outline, holes or cut-outs redrawn
Changed lines of the file:
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@@
-(kicad_pcb (version 20171130) (host pcbnew "(5.0.1)-4")
+(kicad_pcb (version 20171130) (host pcbnew "(5.1.4)-1")
   (general
     (thickness 1.6)
@@
     (zone_45_only no)
     (trace_min 0.2)
-    (segment_width 0.2)
-    (edge_width 0.05)
     (via_size 0.8)
     (via_drill 0.4)
@@
     (uvia_min_size 0.2)
     (uvia_min_drill 0.1)
+    (edge_width 0.05)
+    (segment_width 0.2)
     (pcb_text_width 0.3)
     (pcb_text_size 1.5 1.5)
@@
     (solder_mask_min_width 0.25)
     (aux_axis_origin 0 0)
-    (visible_elements 7FFFFFFF)
+    (visible_elements 7FFFF7FF)
     (pcbplotparams
       (layerselection 0x010fc_ffffffff)
@@
   (gr_line (start 222.25 34.29) (end 222.25 31.75) (layer Edge.Cuts) (width 0.05))
   (gr_line (start 222.25 36.83) (end 222.25 34.29) (layer Edge.Cuts) (width 0.05))
-  (gr_circle (center 218.154 40.894) (end 220.154 40.894) (layer Edge.Cuts) (width 0.05))
+  (gr_circle (center 218.154 35.782) (end 220.154 35.782) (layer Edge.Cuts) (width 0.05))
   (gr_circle (center 70.104 120.396) (end 72.104 120.396) (layer Edge.Cuts) (width 0.05))
-  (gr_circle (center 70.072 40.894) (end 72.072 40.894) (layer Edge.Cuts) (width 0.05))
+  (gr_circle (center 70.072 35.909) (end 72.072 35.909) (layer Edge.Cuts) (width 0.05))
   (gr_circle (center 218.154 120.364) (end 220.154 120.364) (layer Edge.Cuts) (width 0.05))
   (gr_line (start 222.25 36.83) (end 222.25 39.37) (layer Edge.Cuts) (width 0.05))
@@
   (gr_line (start 222.25 121.92) (end 222.25 124.46) (layer Edge.Cuts) (width 0.05))
   (gr_line (start 222.25 39.37) (end 222.25 121.92) (layer Edge.Cuts) (width 0.05))
-  (via (at 166.497 106.807) (size 0.8) (drill 0.4) (layers F.Cu B.Cu) (net 5))
-  (via (at 175.26 109.855) (size 0.8) (drill 0.4) (layers F.Cu B.Cu) (net 5))
-  (via (at 159.766 106.807) (size 0.8) (drill 0.4) (layers F.Cu B.Cu) (net 5))
   (segment (start 120.65 111.07) (end 120.65 109.22) (width 0.25) (layer F.Cu) (net 1))
   (segment (start 117.674 114.046) (end 120.65 111.07) (width 0.25) (layer F.Cu) (net 1))
@@
   (segment (start 148.971 107.442) (end 148.971 101.854) (width 0.25) (layer B.Cu) (net 4))
   (segment (start 148.971 101.854) (end 152.559001 98.265999) (width 0.25) (layer B.Cu) (net 4))
+  (via (at 166.497 106.807) (size 0.8) (drill 0.4) (layers F.Cu B.Cu) (net 5))
+  (via (at 175.26 109.855) (size 0.8) (drill 0.4) (layers F.Cu B.Cu) (net 5))
+  (via (at 159.766 106.807) (size 0.8) (drill 0.4) (layers F.Cu B.Cu) (net 5))
   (segment (start 147.34 86.34) (end 143.51 90.17) (width 0.25) (layer B.Cu) (net 5))
   (segment (start 147.34 67.35) (end 147.34 86.34) (width 0.25) (layer B.Cu) (net 5))
